Commit message: day7초기 코드

File: mastering_ros_robot_description_pkg/urdf/seven_dof_arm.xacro (robot description, xacro)
@@ -144,5 +144,5 @@
   </link>
   <gazebo reference="shoulder_pan_link">
-    <material>Gazebo/Red</material>
+    <material>Gazebo/Blue</material>
   </gazebo>
   <joint name="shoulder_pitch_joint" type="revolute">
@@ -231,5 +231,5 @@
   </link>
   <gazebo reference="elbow_pitch_link">
-    <material>Gazebo/Red</material>
+    <material>Gazebo/Blue</material>
   </gazebo>
   <joint name="wrist_roll_joint" type="revolute">

File: mastering_ros_robot_description_pkg/urdf/seven_dof_arm_with_rgbd.xacro (robot description, xacro)
@@ -145,5 +145,5 @@
   </link>
   <gazebo reference="shoulder_pan_link">
-    <material>Gazebo/Red</material>
+    <material>Gazebo/Blue</material>
   </gazebo>
   <joint name="shoulder_pitch_joint" type="revolute">
